File: pcb/nanoSwinSidC.kicad_pcb (KiCad board)
At the start: 2 copper layers, 35.8 x 17.5 mm, 15 parts, among them J1 Conn_02x03_Odd_Even, J2 Conn_02x14_Counter_Clockwise, U1 ATmega88PA-AU, X1 32 MHz

Commit message: improve pcb layout
Parts:
- moved C2 8.22 mm to (150.1, 97.1), turned to 270 degrees
- moved C3 8.22 mm to (148.6, 97.1), turned to 270 degrees
- moved R4 4.52 mm to (150.6, 88.9), turned to 270 degrees
- moved C1 4.50 mm to (148.6, 93.0)
- moved R6 4.50 mm to (150.1, 93.0), turned to 270 degrees
- moved R2 4.32 mm to (149.1, 88.9)
- moved R1 1.50 mm to (146.1, 88.9)
- moved R3 1.50 mm to (147.6, 88.9)
- turned D1 to 0 degrees
- turned X1 to 270 degrees
Routing:
- net GND: track 75.2 -> 59.7 mm, vias 3 -> 0
- net +5V: track 58.5 -> 69.6 mm, vias 4 -> 2
- net Net-(U1-Pad7): track 24.6 -> 15.2 mm
- net SND: track 22.0 -> 15.9 mm
- net Net-(C1-Pad1): track 10.6 -> 6.69 mm
- net Net-(D1-Pad1): track 7.41 -> 4.37 mm
- net SCK: track 37.7 -> 34.8 mm
- net nRST: track 54.3 -> 52.2 mm
- net Net-(R2-Pad2): track 3.21 -> 5.21 mm
- net nCS: track 19.9 -> 21.8 mm, vias 1 -> 2
- net A1: track 14.1 -> 15.6 mm
- net Net-(R4-Pad2): track 4.89 -> 3.88 mm
- net D7: track 13.1 -> 12.2 mm
- net A0: track 13.9 -> 14.7 mm
- net A2: track 13.9 -> 13.4 mm
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Other:
- board text added: "6581"
- board text added: "SwinSID"
- board text added: "nano"
- board text removed: "SwinSID Nano"

Commit message: add derived files
Other:
- board text added: "AVR ISP"
- board text added: "JLCJLCJLCJLC"
Changed lines of the file:
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@@
   (general
     (thickness 1.6)
-    (drawings 12)
+    (drawings 14)
     (tracks 301)
     (zones 0)
@@
     (46 B.CrtYd user)
     (47 F.CrtYd user)
-    (48 B.Fab user hide)
-    (49 F.Fab user hide)
+    (48 B.Fab user)
+    (49 F.Fab user)
   )
   (setup
@@
     (visible_elements 7FFFFF7F)
     (pcbplotparams
-      (layerselection 0x010fc_ffffffff)
+      (layerselection 0x010f0_ffffffff)
       (usegerberextensions false)
       (usegerberattributes false)
@@
       (psa4output false)
       (plotreference true)
-      (plotvalue true)
+      (plotvalue false)
       (plotinvisibletext false)
       (padsonsilk false)
@@
       (outputformat 1)
       (mirror false)
-      (drillshape 1)
+      (drillshape 0)
       (scaleselection 1)
-      (outputdirectory ""))
+      (outputdirectory "out/gerber/"))
   )
   (net 0 "")
@@
       (effects (font (size 0.7 1) (thickness 0.15)) (justify mirror))
     )
-    (fp_text value 2.2k (at -1.675 0.7) (layer B.Fab)
+    (fp_text value 2.2k (at -1.775 0.8) (layer B.Fab)
       (effects (font (size 1 1) (thickness 0.15)) (justify mirror))
     )
@@
       (effects (font (size 0.7 1) (thickness 0.15)) (justify mirror))
     )
-    (fp_text value "32 MHz" (at 4.5 0 180) (layer B.Fab)
+    (fp_text value "32 MHz" (at -4.7 0 180) (layer B.Fab)
       (effects (font (size 1 1) (thickness 0.15)) (justify mirror))
     )
@@
       (effects (font (size 0.7 1) (thickness 0.15)) (justify mirror))
     )
-    (fp_text value 1k (at -1.675 0.9 180) (layer B.Fab)
+    (fp_text value 1k (at 1.875 -2.2 180) (layer B.Fab)
       (effects (font (size 1 1) (thickness 0.15)) (justify mirror))
     )
@@
       (effects (font (size 0.7 1) (thickness 0.15)) (justify mirror))
     )
-    (fp_text value 1k (at 1.575 0.9) (layer B.Fab)
+    (fp_text value 1k (at 1.875 0.9) (layer B.Fab)
       (effects (font (size 1 1) (thickness 0.15)) (justify mirror))
     )
@@
       (effects (font (size 0.7 1) (thickness 0.15)) (justify mirror))
     )
-    (fp_text value 240k (at -2.275 0.1) (layer B.Fab)
+    (fp_text value 240k (at -1.775 -2.4) (layer B.Fab)
       (effects (font (size 1 1) (thickness 0.15)) (justify mirror))
     )
@@
       (effects (font (size 0.7 1) (thickness 0.15)) (justify mirror))
     )
-    (fp_text value 1k (at 1.675 -1.4 180) (layer B.Fab)
+    (fp_text value 1k (at -1.775 -0.7 180) (layer B.Fab)
       (effects (font (size 1 1) (thickness 0.15)) (justify mirror))
     )
@@
       (effects (font (size 0.7 1) (thickness 0.15)) (justify mirror))
     )
-    (fp_text value 4.7k (at -1.725 -0.1) (layer B.Fab)
+    (fp_text value 4.7k (at 1.775 -3) (layer B.Fab)
       (effects (font (size 1 1) (thickness 0.15)) (justify mirror))
     )
@@
       (effects (font (size 0.7 1) (thickness 0.15)) (justify mirror))
     )
-    (fp_text value 10n (at 1.675 0 180) (layer B.Fab)
+    (fp_text value 10n (at 2.225 1.4 180) (layer B.Fab)
       (effects (font (size 1 1) (thickness 0.15)) (justify mirror))
     )
@@
       (effects (font (size 0.7 1) (thickness 0.15)) (justify mirror))
     )
-    (fp_text value 100n (at -1.625 0.9 180) (layer B.Fab)
+    (fp_text value 100n (at 2.325 -1.1 180) (layer B.Fab)
       (effects (font (size 1 1) (thickness 0.15)) (justify mirror))
     )
@@
       (effects (font (size 0.7 1) (thickness 0.15)) (justify mirror))
     )
-    (fp_text value 470p (at 1.775 0.9) (layer B.Fab)
+    (fp_text value 470p (at 1.875 -0.7) (layer B.Fab)
       (effects (font (size 1 1) (thickness 0.15)) (justify mirror))
     )
@@
     )
   )
+  (gr_text "AVR ISP" (at 139.8 93.3) (layer F.Fab)
+    (effects (font (size 1 1) (thickness 0.15)))
+  )
+  (gr_text JLCJLCJLCJLC (at 157.3 99.2) (layer B.SilkS)
+    (effects (font (size 0.8 0.8) (thickness 0.15)) (justify mirror))
+  )
   (gr_text nano (at 151.8 95.1) (layer F.SilkS)
